File: BSPD_v2/BSPD_V2.kicad_pcb (KiCad board)
At the start: 2 copper layers, 85.5 x 52 mm, 0 parts

Commit message: Updated pcb design
Parts:
- added C1: C_Generic, Capacitor_THT:C_Disc_D12.5mm_W5.0mm_P10.00mm, F.Cu at (107.5, 86.5)
- added C2: C_Generic, Capacitor_THT:C_Disc_D12.5mm_W5.0mm_P10.00mm, F.Cu at (115.0, 119.5)
- added D1: LED, LED_THT:LED_D5.0mm_Horizontal_O6.35mm_Z9.0mm, F.Cu at (152.7, 130.5)
- added D2: LED, LED_THT:LED_D5.0mm_Horizontal_O6.35mm_Z9.0mm, F.Cu at (160.2, 130.5)
- added D3: LED, LED_THT:LED_D5.0mm_Horizontal_O6.35mm_Z9.0mm, F.Cu at (167.7, 130.5)
- added K1: G5V-1, Relay_THT:Relay_SPDT_Omron_G5V-1, F.Cu at (133.6, 64.0)
- added P1: 0430450827, Connector_Molex:Molex_Mega-Fit_76825-0008_2x04_P5.70mm_Horizontal, F.Cu at (158.8, 105.5)
- added R1: R, PCM_Resistor_THT_AKL:R_Axial_DIN0204_L3.6mm_D1.6mm_P2.54mm_Vertical, F.Cu at (108.3, 77.5)
- added R2: R, PCM_Resistor_THT_AKL:R_Axial_DIN0204_L3.6mm_D1.6mm_P2.54mm_Vertical, F.Cu at (107.8, 109.5)
- added R3: R, PCM_Resistor_THT_AKL:R_Axial_DIN0204_L3.6mm_D1.6mm_P2.54mm_Vertical, F.Cu at (167.8, 125.0)
- added R4: R, PCM_Resistor_THT_AKL:R_Axial_DIN0204_L3.6mm_D1.6mm_P2.54mm_Vertical, F.Cu at (160.5, 125.0)
- added R5: R, PCM_Resistor_THT_AKL:R_Axial_DIN0204_L3.6mm_D1.6mm_P2.54mm_Vertical, F.Cu at (152.3, 125.0)
- added S1: EG1206, Button_Switch_THT:SW_E-Switch_EG1224_SPDT_Angled, F.Cu at (163.0, 71.0)
- added T1: T-BJT-NPN, PCM_Package_TO_SOT_THT_AKL_OneLayer:TO-92L_ECB, F.Cu at (122.7, 70.3)
- added TRIM1: TrimPot_TC33X_1k, PCM_Potentiometer_THT_AKL_Double:Potentiometer_Bourns_3296W_Vertical, F.Cu at (80.0, 82.0)
- added TRIM2: TrimPot_T73YEt_1k, PCM_Potentiometer_THT_AKL_Double:Potentiometer_Bourns_3296W_Vertical, F.Cu at (80.5, 103.5)
- added TRIM3: TrimPot_T73YEt_1k, PCM_Potentiometer_THT_AKL_Double:Potentiometer_Bourns_3296W_Vertical, F.Cu at (80.5, 93.0)
- added TRIM4: TrimPot_T73YEt_10k, PCM_Potentiometer_THT_AKL_Double:Potentiometer_Bourns_3296W_Vertical, F.Cu at (99.1, 82.0)
- added TRIM5: TrimPot_T73YEt_10k, PCM_Potentiometer_THT_AKL_Double:Potentiometer_Bourns_3296W_Vertical, F.Cu at (98.5, 90.5)
- added U1: SN74HC00N, PCM_4ms_Package_DIP:DIP-14_W7.62mm, F.Cu at (93.5, 72.3)
- added U2: LM393P, PCM_4ms_Package_DIP:DIP-8pin_TH, F.Cu at (74.2, 63.9)
- added U3: LM393P, PCM_4ms_Package_DIP:DIP-8pin_TH, F.Cu at (74.4, 113.5)
- added U4: LM393P, PCM_Package_DIP_AKL:DIP-8_W7.62mm, F.Cu at (96.5, 115.9)
- added U5: SN74HC08N, PCM_4ms_Package_DIP:DIP-14_W7.62mm, F.Cu at (94.0, 104.3)
- added U6: LM2596T-5, PCM_Package_TO_SOT_THT_AKL:TO-220F-5_P3.4x2.06mm_StaggerEven_Lead1.86mm_Vertical, F.Cu at (149.0, 64.6)
Other:
- board size 85.5 x 52 mm -> 118 x 85.5 mm

Commit message: Updated pcb design with check
Routing:
- net GND: track 0.00 -> 318.8 mm
- net TPS_sensor: track 0.00 -> 137.7 mm, vias 0 -> 1
- net +5V: track 0.00 -> 120.5 mm
- net BPS_sensor: track 0.00 -> 120.4 mm
- net Net-(U6-OUT): track 0.00 -> 68.4 mm
- net Net-(U1-1B): track 0.00 -> 57.4 mm, vias 0 -> 1
- net Net-(TRIM3-Center): track 0.00 -> 54.2 mm, vias 0 -> 1
- net Net-(U4-1IN-): track 0.00 -> 52.2 mm, vias 0 -> 1
- net Net-(T1-B): track 0.00 -> 45.4 mm
- net Net-(U2-2OUT): track 0.00 -> 42.8 mm
- net Net-(TRIM4-Center): track 0.00 -> 41.3 mm
- net Net-(TRIM5-Center): track 0.00 -> 36.5 mm
- net Net-(U4-2IN-): track 0.00 -> 24.7 mm
- net Net-(U1-1A): track 0.00 -> 22.7 mm
- net Net-(U3-2OUT): track 0.00 -> 19.7 mm
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
Commit message: pcb design updated using proper footprints and routing
Parts:
- moved D1 12.3 mm to (147.2, 119.5)
- moved D2 12.3 mm to (154.7, 119.5)
- moved D3 12.3 mm to (162.2, 119.5)
- moved R3 12.3 mm to (162.3, 114.0)
- moved R4 12.3 mm to (155.0, 114.0)
- moved R5 12.3 mm to (146.8, 114.0)
Routing:
- net BPS_sensor: track 120.4 -> 103.0 mm
- net GND: track 318.8 -> 308.7 mm
- net Net-(U6-OUT): track 68.4 -> 59.7 mm
- net TPS_sensor: track 137.7 -> 129.7 mm
Other:
- board size 118 x 85.5 mm -> 109.5 x 81.5 mm
Changed lines of the file:
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@@
 	(footprint "PCM_Resistor_THT_AKL:R_Axial_DIN0204_L3.6mm_D1.6mm_P2.54mm_Vertical"
 		(layer "F.Cu")
-		(at 160.5 125)
+		(at 155 114.025)
 		(descr "Resistor, Axial_DIN0204 series, Axial, Vertical, pin pitch=2.54mm, 0.167W, length*diameter=3.6*1.6mm^2, http://cdn-reichelt.de/documents/datenblatt/B400/1_4W%23YAG.pdf")
 		(tags "Resistor Axial_DIN0204 series Axial Vertical pin pitch 2.54mm 0.167W length 3.6mm diameter 1.6mm")
@@
 	(footprint "LED_THT:LED_D5.0mm_Horizontal_O6.35mm_Z9.0mm"
 		(layer "F.Cu")
-		(at 167.705 130.475)
+		(at 162.205 119.5)
 		(descr "LED, diameter 5.0mm, horizontal offset 6.35mm, z-position of LED center 9.0mm, 2 pins, generated by kicad-footprint-generator")
 		(tags "LED")
@@
 	(footprint "PCM_Resistor_THT_AKL:R_Axial_DIN0204_L3.6mm_D1.6mm_P2.54mm_Vertical"
 		(layer "F.Cu")
-		(at 167.78 125)
+		(at 162.28 114.025)
 		(descr "Resistor, Axial_DIN0204 series, Axial, Vertical, pin pitch=2.54mm, 0.167W, length*diameter=3.6*1.6mm^2, http://cdn-reichelt.de/documents/datenblatt/B400/1_4W%23YAG.pdf")
 		(tags "Resistor Axial_DIN0204 series Axial Vertical pin pitch 2.54mm 0.167W length 3.6mm diameter 1.6mm")
@@
 	(footprint "LED_THT:LED_D5.0mm_Horizontal_O6.35mm_Z9.0mm"
 		(layer "F.Cu")
-		(at 152.745 130.475)
+		(at 147.245 119.5)
 		(descr "LED, diameter 5.0mm, horizontal offset 6.35mm, z-position of LED center 9.0mm, 2 pins, generated by kicad-footprint-generator")
 		(tags "LED")
@@
 	(footprint "LED_THT:LED_D5.0mm_Horizontal_O6.35mm_Z9.0mm"
 		(layer "F.Cu")
-		(at 160.225 130.475)
+		(at 154.725 119.5)
 		(descr "LED, diameter 5.0mm, horizontal offset 6.35mm, z-position of LED center 9.0mm, 2 pins, generated by kicad-footprint-generator")
 		(tags "LED")
@@
 	(footprint "PCM_Resistor_THT_AKL:R_Axial_DIN0204_L3.6mm_D1.6mm_P2.54mm_Vertical"
 		(layer "F.Cu")
-		(at 152.28 125)
+		(at 146.78 114.025)
 		(descr "Resistor, Axial_DIN0204 series, Axial, Vertical, pin pitch=2.54mm, 0.167W, length*diameter=3.6*1.6mm^2, http://cdn-reichelt.de/documents/datenblatt/B400/1_4W%23YAG.pdf")
 		(tags "Resistor Axial_DIN0204 series Axial Vertical pin pitch 2.54mm 0.167W length 3.6mm diameter 1.6mm")
@@
 	)
 	(gr_rect
-		(start 56.95 50.31)
-		(end 174.95 135.81)
+		(start 67.5 55.5)
+		(end 177 137)
 		(stroke
 			(width 0.05)
@@
 	)
 	(segment
-		(start 159.0233 131.6767)
-		(end 159.0233 130.475)
+		(start 153.5233 120.7017)
+		(end 153.5233 119.5)
 		(width 0.2)
 		(layer "F.Cu")
@@
 	)
 	(segment
-		(start 140.5683 119.5)
-		(end 125 119.5)
-		(width 0.2)
-		(layer "F.Cu")
-		(net 1)
-	)
-	(segment
 		(start 111.7717 70.27)
 		(end 109.7417 72.3)
@@
 	)
 	(segment
-		(start 152.745 130.475)
-		(end 153.9467 130.475)
+		(start 147.245 119.5)
+		(end 148.4467 119.5)
 		(width 0.2)
 		(layer "F.Cu")
@@
 	)
 	(segment
-		(start 167.705 130.475)
-		(end 166.5033 130.475)
+		(start 162.205 119.5)
+		(end 161.0033 119.5)
 		(width 0.2)
 		(layer "F.Cu")
@@
 	)
 	(segment
-		(start 151.5433 130.475)
-		(end 140.5683 119.5)
+		(start 125 119.5)
+		(end 147.245 119.5)
 		(width 0.2)
 		(layer "F.Cu")
@@
 	)
 	(segment
-		(start 154.7729 131.6767)
-		(end 159.0233 131.6767)
+		(start 149.2729 120.7017)
+		(end 153.5233 120.7017)
 		(width 0.2)
 		(layer "F.Cu")
@@
 	)
 	(segment
-		(start 159.0233 131.6767)
-		(end 165.3016 131.6767)
+		(start 153.5233 120.7017)
+		(end 159.8016 120.7017)
 		(width 0.2)
 		(layer "F.Cu")
@@
 	)
 	(segment
-		(start 165.3016 131.6767)
-		(end 166.5033 130.475)
+		(start 159.8016 120.7017)
+		(end 161.0033 119.5)
 		(width 0.2)
 		(layer "F.Cu")
@@
 	)
 	(segment
-		(start 160.225 130.475)
-		(end 159.0233 130.475)
+		(start 154.725 119.5)
+		(end 153.5233 119.5)
 		(width 0.2)
 		(layer "F.Cu")
@@
 	)
 	(segment
-		(start 153.9467 130.8505)
-		(end 154.7729 131.6767)
+		(start 148.4467 119.8755)
+		(end 149.2729 120.7017)
 		(width 0.2)
 		(layer "F.Cu")
@@
 	)
 	(segment
-		(start 153.9467 130.475)
-		(end 153.9467 130.8505)
+		(start 148.4467 119.5)
+		(end 148.4467 119.8755)
 		(width 0.2)
 		(layer "F.Cu")
@@
 	)
 	(segment
-		(start 152.745 130.475)
-		(end 151.5433 130.475)
-		(width 0.2)
-		(layer "F.Cu")
-		(net 1)
-	)
-	(segment
 		(start 96.5 123.54)
 		(end 97.6017 123.54)
@@
 	)
 	(segment
-		(start 152.28 125)
-		(end 155.285 128.005)
+		(start 146.78 114.025)
+		(end 149.785 117.03)
 		(width 0.2)
 		(layer "B.Cu")
@@
 	)
 	(segment
-		(start 155.285 128.005)
-		(end 155.285 130.475)
+		(start 149.785 117.03)
+		(end 149.785 119.5)
 		(width 0.2)
 		(layer "B.Cu")
@@
 	)
 	(segment
-		(start 162.765 127.265)
-		(end 160.5 125)
+		(start 157.265 116.29)
+		(end 155 114.025)
 		(width 0.2)
 		(layer "B.Cu")
@@
 	)
 	(segment
-		(start 162.765 130.475)
-		(end 162.765 127.265)
+		(start 157.265 119.5)
+		(end 157.265 116.29)
 		(width 0.2)
 		(layer "B.Cu")
@@
 	)
 	(segment
-		(start 167.78 125)
-		(end 170.245 127.465)
+		(start 162.28 114.025)
+		(end 164.745 116.49)
 		(width 0.2)
 		(layer "B.Cu")
@@
 	)
 	(segment
-		(start 170.245 127.465)
-		(end 170.245 130.475)
+		(start 164.745 116.49)
+		(end 164.745 119.5)
 		(width 0.2)
 		(layer "B.Cu")
@@
 	(segment
 		(start 158.775 105.55)
-		(end 154.82 109.505)
+		(end 154.9125 109.4125)
+		(width 0.2)
+		(layer "B.Cu")
+		(net 11)
+	)
+	(segment
+		(start 153.9325 109.4125)
+		(end 154.9125 109.4125)
 		(width 0.2)
 		(layer "B.Cu")
@@
 	)
 	(segment
+		(start 149.32 114.025)
+		(end 153.9325 109.4125)
+		(width 0.2)
+		(layer "B.Cu")
+		(net 11)
+	)
+	(segment
 		(start 83.2498 97.2975)
 		(end 83.2498 71.3132)
@@
 	)
 	(segment
-		(start 82.0383 70.1017)
-		(end 81.81 70.1017)
+		(start 154.9125 109.4125)
+		(end 154.82 109.505)
 		(width 0.2)
 		(layer "B.Cu")
@@
 	)
 	(segment
-		(start 81.81 69)
+		(start 82.0383 70.1017)
 		(end 81.81 70.1017)
 		(width 0.2)
@@
 	)
 	(segment
-		(start 154.82 109.505)
-		(end 154.82 125)
+		(start 81.81 69)
+		(end 81.81 70.1017)
 		(width 0.2)
 		(layer "B.Cu")
@@
 	)
 	(segment
-		(start 84.5003 117.1814)
-		(end 83.1017 118.58)
+		(start 74.38 116.04)
+		(end 75.4817 116.04)
 		(width 0.2)
 		(layer "F.Cu")
@@
 	)
 	(segment
-		(start 82 118.58)
-		(end 83.1017 118.58)
+		(start 157.1564 114.025)
+		(end 157.54 114.025)
 		(width 0.2)
 		(layer "F.Cu")
@@
 	)
 	(segment
-		(start 74.38 116.04)
-		(end 75.4817 116.04)
+		(start 75.4817 116.04)
+		(end 78.0217 118.58)
 		(width 0.2)
 		(layer "F.Cu")
@@
 	)
 	(segment
-		(start 75.4817 116.04)
-		(end 78.0217 118.58)
+		(start 154 117.1814)
+		(end 157.1564 114.025)
 		(width 0.2)
 		(layer "F.Cu")
@@
 	)
 	(segment
-		(start 154.2197 117.1814)
-		(end 84.5003 117.1814)
+		(start 82 118.58)
+		(end 83.1017 118.58)
 		(width 0.2)
 		(layer "F.Cu")
@@
 	)
 	(segment
-		(start 162.0383 125)
-		(end 154.2197 117.1814)
+		(start 83.1017 118.58)
+		(end 84.5003 117.1814)
 		(width 0.2)
 		(layer "F.Cu")
@@
 	)
 	(segment
-		(start 163.04 125)
-		(end 162.0383 125)
+		(start 84.5003 117.1814)
+		(end 154 117.1814)
 		(width 0.2)
 		(layer "F.Cu")
@@
 	)
 	(segment
-		(start 158.775 99.85)
-		(end 161.5002 102.5752)
+		(start 157.54 114.025)
+		(end 161.4625 110.1025)
 		(width 0.2)
 		(layer "B.Cu")
@@
 	)
 	(segment
-		(start 163.04 125)
-		(end 163.04 123.9983)
+		(start 161.4625 102.5375)
+		(end 158.775 99.85)
 		(width 0.2)
 		(layer "B.Cu")
@@
 	)
 	(segment
-		(start 161.5002 122.4585)
-		(end 163.04 123.9983)
+		(start 161.4625 110.1025)
+		(end 161.4625 102.5375)
 		(width 0.2)
 		(layer "B.Cu")
@@
 	)
 	(segment
-		(start 161.5002 102.5752)
-		(end 161.5002 122.4585)
+		(start 170.32 108.525)
+		(end 170.32 107.5)
 		(width 0.2)
 		(layer "B.Cu")
-		(net 12)
+		(net 16)
+	)
+	(segment
+		(start 170.32 94.495)
+		(end 170.32 107.5)
+		(width 0.2)
+		(layer "B.Cu")
+		(net 16)
 	)
 	(segment
@@
 	)
 	(segment
+		(start 164.82 114.025)
+		(end 170.32 108.525)
+		(width 0.2)
+		(layer "B.Cu")
+		(net 16)
+	)
+	(segment
 		(start 148.9973 69.7)
 		(end 149.093 69.7)
@@
 	)
 	(segment
-		(start 170.32 94.495)
-		(end 170.32 125)
-		(width 0.2)
-		(layer "B.Cu")
-		(net 16)
-	)
-	(segment
 		(start 98.48 72.3)
 		(end 99.5817 72.3)
@@
 		(min_thickness 0.25)
 		(filled_areas_thickness no)
-		(fill yes
+		(fill
 			(thermal_gap 0.5)
 			(thermal_bridge_width 0.5)
@@
 		(polygon
 			(pts
-				(xy 57.45 50.81) (xy 174.45 50.81) (xy 174.45 135.31) (xy 57.45 135.31)
+				(xy 68.45 56.31) (xy 176.45 56.31) (xy 176.45 136.31) (xy 68.45 136.31)
 			)
 		)

Commit message: Added footprints for 5v Regulator
Parts:
- removed K1: G5V-1, Relay_THT:Relay_SPDT_Omron_G5V-1
- added D4: LED, LED_THT:LED_D5.0mm_Horizontal_O6.35mm_Z9.0mm, F.Cu at (154.2, 120.5)
- added K2: SR1-5V-450-1C, SR1-5V-450-1C:RELAY_SR1-5V-450-1C, F.Cu at (126.0, 68.5)
- added R6: R, PCM_Resistor_THT_AKL:R_Axial_DIN0204_L3.6mm_D1.6mm_P2.54mm_Vertical, F.Cu at (154.0, 115.0)
- U2, U3: footprint PCM_4ms_Package_DIP:DIP-8pin_TH -> PCM_Package_DIP_AKL:DIP-8_W7.62mm
- moved D1 15.5 mm to (131.7, 120.5)
- moved D2 15.5 mm to (139.2, 120.5)
- moved D3 15.5 mm to (146.7, 120.5)
- moved R3 15.5 mm to (146.8, 115.0)
- moved R4 15.5 mm to (139.5, 115.0)
- moved R5 15.5 mm to (131.3, 115.0)
- moved S1 10.7 mm to (152.3, 71.5)
- moved U6 10.7 mm to (138.3, 65.1)
- moved P1 10.5 mm to (148.3, 106.1)
- moved T1 8.82 mm to (126.0, 78.5)
Connections:
- P1 pad 6: unconnected-(P1-Pad6) -> E_ON
- P1 pad 7: unconnected-(P1-Pad7) -> OUT
Routing:
- net E_ON: track 0.00 -> 75.8 mm, vias 0 -> 1
- net OUT: track 5.08 -> 46.4 mm, vias 0 -> 1
- net GND: track 308.7 -> 286.8 mm, vias 0 -> 1
- net BPS_sensor: track 103.0 -> 88.2 mm
- net TPS_sensor: track 129.7 -> 116.4 mm
- net Net-(D4-A): track 0.00 -> 6.64 mm
- net +5V: track 120.5 -> 123.3 mm
- net Net-(T1-B): track 45.4 -> 42.6 mm, vias 0 -> 1
- net Net-(U6-OUT): track 59.7 -> 57.8 mm
- net Net-(U4-1IN-): track 52.2 -> 51.0 mm
- net Net-(T1-E): track 13.5 -> 12.5 mm
- net Net-(TRIM4-Center): track 41.3 -> 40.4 mm
- net Net-(U1-1Y): track 15.5 -> 14.6 mm
Other:
- board size 109.5 x 81.5 mm -> 95.5 x 81.5 mm
